Commit message: URDF rebuild, joint states msgs does not published in rviz

File: Monster_Truck_URDF/urdf/Monster_Truck.xacro (robot description, xacro)
@@ -6,16 +6,12 @@
                 <color rgba="0 0 1 1"/>
             </material>
-            <origin rpy="0 0 0" xyz="0 0 0.3"/>
+            <origin rpy="0 0 0" xyz="0 0 0.2"/>
             <geometry>
-                <box size="2 0.5 0.3"/>
+                <box size="1 0.5 0.1"/>
             </geometry>
         </visual>
     </link>
-    <joint name="front" type="fixed">
-        <axis xyz="0 0 1" />
-        <origin rpy="0 0 0" xyz="0 0 0"/>
-        <parent link="base_link"/>
-        <child link="front"/>
-    </joint>
+<!--****************************************-->
+<!--****************************************-->
     <link name="front">
         <visual>
@@ -23,5 +19,5 @@
                 <color rgba="0 0 0 1"/>
             </material>
-            <origin rpy="0 0 0" xyz="-1 0 0.4"/>
+            <origin rpy="0 0 0" xyz="0 0.5 0.25"/>
             <geometry>
                 <box size="0.1 0.1 0.2"/>
@@ -29,171 +25,89 @@
         </visual>
     </link>
-    <!--Links for connect wheels and base link-->
-    <joint name="fixed_back_left" type="fixed">
-        <axis xyz="0 0 1" />
-        <origin rpy="0 0 0" xyz="0 0 0"/>
-        <parent link="base_link"/>
-        <child link="connect_left_back_wheel"/>
-    </joint>
-    <link name="connect_left_back_wheel">
+  <joint name="front_joint" type="fixed">
+    <parent link="base_link"/>
+    <child link="front"/>
+    <origin xyz="0 0 0" rpy="0 0 0"/>
+    <axis xyz="1 0 0"/>
+  </joint>
+<!--****************************************-->
+<!--****************************************-->
+    <link name="link_left_f">
         <visual>
-            <material name="Black">
-                <color rgba="0 0 0 1"/>
+            <material name="Red">
+                <color rgba="1 0 0 1"/>
             </material>
-            <origin rpy="0 0 0" xyz="0.5 -0.1 0.1"/>
+            <origin rpy="0 0 0" xyz="-0.3 0.1 0.1"/>
             <geometry>
-                <box size="0.2 0.15 0.2"/>
+                <box size="0.05 0.05 0.1"/>
             </geometry>
         </visual>
     </link>
-    <joint name="fixed_front_left" type="fixed">
-        <axis xyz="0 0 1" />
-        <origin rpy="0 0 0" xyz="0 0 0"/>
-        <parent link="base_link"/>
-        <child link="connect_left_front_wheel"/>
-    </joint>
-    <link name="connect_left_front_wheel">
+  <joint name="fixed_left_front" type="fixed">
+    <parent link="base_link"/>
+    <child link="link_left_f"/>
+    <origin xyz="0 0 0" rpy="0 0 0"/>
+    <axis xyz="0 0 0"/>
+  </joint>
+<!--****************************************-->
+<!--****************************************-->
+    <link name="link_left_f_2">
         <visual>
-            <material name="Black">
-                <color rgba="0 0 0 1"/>
+            <material name="Green">
+                <color rgba="0 1 0 1"/>
             </material>
-            <origin rpy="0 0 0" xyz="-0.5 -0.1 0.1"/>
+            <origin rpy="0 0 0" xyz="-0.2 0.2 0.05"/>
             <geometry>
-                <box size="0.2 0.15 0.2"/>
+                <box size="0.05 0.2 0.05"/>
             </geometry>
         </visual>
     </link>
-    <!--Links for connect wheels and base link-->
-    <joint name="fixed_back_right" type="fixed">
-        <axis xyz="0 0 1" />
-        <origin rpy="0 0 0" xyz="0 0 0"/>
-        <parent link="base_link"/>
-        <child link="connect_right_back_wheel"/>
-    </joint>
-    <link name="connect_right_back_wheel">
+  <joint name="fixed_left_front_2" type="fixed">
+    <parent link="link_left_f"/>
+    <child link="link_left_f_2"/>
+    <origin xyz="0 0 0" rpy="0 0 0"/>
+    <axis xyz="0 0 0"/>
+  </joint>
+<!--****************************************-->
+<!--****************************************-->
+  <link name="left_wheel_f">
         <visual>
-            <material name="Black">
+   	        <material name="Black">
                 <color rgba="0 0 0 1"/>
             </material>
-            <origin rpy="0 0 0" xyz="0.5 0.1 0.1"/>
+             <origin xyz="0 0 0" rpy="1.570795 0 0" />
             <geometry>
-                <box size="0.2 0.15 0.2"/>
+                <cylinder length="0.15" radius="0.12" />
             </geometry>
         </visual>
     </link>
-    <joint name="fixed_front_right" type="fixed">
-        <axis xyz="0 0 1" />
-        <origin rpy="0 0 0" xyz="0 0 0"/>
-        <parent link="base_link"/>
-        <child link="connect_right_front_wheel"/>
-    </joint>
-    <link name="connect_right_front_wheel">
+<!--****************************************-->
+<!--****************************************-->
+  <joint name="joint_left_wheel_f" type="continuous">
+    <parent link="link_left_f_2"/>
+    <child link="left_wheel_f"/>
+    <origin xyz="-0.20 0.30 0" rpy="0 0 0" />
+    <axis xyz="0 1 0" />
+    <limit effort="100" velocity="100"/>
+    <joint_properties damping="0.0" friction="0.0"/>
+  </joint>
+<!--****************************************-->
+<!--****************************************-->
+    <link name="sign_left_front">
         <visual>
-            <material name="Black">
-                <color rgba="0 0 0 1"/>
+            <material name="White">
+                <color rgba="1 1 1 1"/>
             </material>
-            <origin rpy="0 0 0" xyz="-0.5 0.1 0.08"/>
+            <origin rpy="0 0 0" xyz="0 0 0.12"/>
             <geometry>
-                <box size="0.2 0.15 0.31"/>
+                <sphere radius="0.02" />
             </geometry>
         </visual>
     </link>
-    <joint name="fixed_front_right_2" type="fixed">
-        <axis xyz="0 0 1" />
-        <origin rpy="0 0 0" xyz="0 0 0"/>
-        <parent link="connect_right_front_wheel"/>
-        <child link="connect_right_front_wheel_2"/>
-    </joint>
-    <link name="connect_right_front_wheel_2">
-        <visual>
-            <material name="Black">
-                <color rgba="0 0 0 1"/>
-            </material>
-            <origin rpy="0 0 0" xyz="-0.5 0.3 0"/>
-            <geometry>
-                <box size="0.2 0.3 0.15"/>
-            </geometry>
-        </visual>
-    </link>
-    <!--Joint for right back wheel-->
-    <joint name="base_link_right_back_wheel" type="continuous">
-        <axis xyz="0 1 0" />
-        <limit effort="1000.0" velocity="0.5" />
-        <origin rpy="0 0 0" xyz="0 0 0.5"/>
-        <parent link="connect_right_front_wheel_2"/>
-        <child link="right_wheel_back"/>
-    </joint>
-    <!--right back wheel-->
-    <link name="right_wheel_back">
-    <visual>
-   	<material name="Black">
-      <color rgba="0 0 1 1"/>
-    </material>
-      <origin xyz="-0.5 0.6 0" rpy="1.570795 0 0" />
-      <geometry>
-          <cylinder length="0.5" radius="0.3" />
-      </geometry>
-    </visual>
-    </link>
-      <!--Joint for left back wheel-->
-    <joint name="base_link_left_back_wheel" type="continuous">
-        <axis xyz="0 1 0" />
-        <limit effort="1000.0" lower="-3.14" upper="3.14" velocity="0.5" />
-        <origin rpy="0 0 0" xyz="0 0 0.5"/>
-        <parent link="base_link"/>
-        <child link="left_wheel_back"/>
-    </joint>
-    <!--left back wheel-->
-    <link name="left_wheel_back">
-    <visual>
-   	<material name="Black">
-      <color rgba="0 0 0 1"/>
-    </material>
-      <origin xyz="-0.5 -0.6 0" rpy="1.570795 0 0" />
-      <geometry>
-          <cylinder length="0.3" radius="0.3" />
-      </geometry>
-    </visual>
-    </link>
-    <!--Joint for right front wheel-->
-    <joint name="base_link_right_front_wheel" type="continuous">
-        <axis xyz="1 0 0" />
-        <limit effort="1000.0" lower="-3.14" upper="3.14" velocity="0.5" />
-        <origin rpy="0 0 0" xyz="0 0 0.5"/>
-        <parent link="base_link"/>
-        <child link="right_wheel_front"/>
-    </joint>
-    <!--right front  wheel-->
-    <link name="right_wheel_front">
-    <visual>
-   	<material name="Black">
-      <color rgba="0 0 0 1"/>
-    </material>
-      <origin xyz="0.5 0.6 0" rpy="1.570795 0 0" />
-      <geometry>
-          <cylinder length="0.3" radius="0.3" />
-      </geometry>
-    </visual>
-    </link>
-      <!--Joint for left front wheel-->
-    <joint name="base_link_left_front_wheel" type="continuous">
-        <axis xyz="0 1 0" />
-        <limit effort="1000.0" velocity="0.5" />
-        <joint_properties damping="0.0" friction="0.0"/>
-        <origin rpy="0 0 0" xyz="0 0 0.5"/>
-        <parent link="base_link"/>
-        <child link="left_wheel_front"/>
-    </joint>
-    <!--left front wheel-->
-    <link name="left_wheel_front">
-    <visual>
-   	<material name="Black">
-      <color rgba="0 0 0 1"/>
-    </material>
-      <origin xyz="0.5 -0.6 0" rpy="1.570795 0 0" />
-      <geometry>
-          <cylinder length="0.3" radius="0.3" />
-      </geometry>
-    </visual>
-    </link>
+  <joint name="fixed_sign_left_f" type="fixed">
+    <parent link="left_wheel_f"/>
+    <child link="sign_left_front"/>
+    <origin xyz="0 0 0" rpy="0 0 0"/>
+    <axis xyz="1 0 0"/>
+  </joint>
 </robot>

Commit message: error when publish tf2_messages

File: Monster_Truck_URDF/urdf/Monster_Truck.xacro (robot description, xacro)
@@ -84,11 +84,11 @@
 <!--****************************************-->
 <!--****************************************-->
-  <joint name="joint_left_wheel_f" type="continuous">
+  <joint name="joint_left_wheel_f" type="revolute">
     <parent link="link_left_f_2"/>
     <child link="left_wheel_f"/>
     <origin xyz="-0.20 0.30 0" rpy="0 0 0" />
     <axis xyz="0 1 0" />
-    <limit effort="100" velocity="100"/>
-    <joint_properties damping="0.0" friction="0.0"/>
+  <dynamics damping="0.7"/>
+  <limit effort="1000" velocity="0.5" lower="-3.14" upper="3.14" />
   </joint>
 <!--****************************************-->

Commit message: URDF implemented, publish jointstates for rviz visualization

File: Monster_Truck_URDF/urdf/Monster_Truck.xacro (robot description, xacro)
@@ -3,10 +3,10 @@
     <link name="base_link">
         <visual>
-            <material name="Blue">
-                <color rgba="0 0 1 1"/>
+            <material name="Black">
+                <color rgba="0 0 0 1"/>
             </material>
             <origin rpy="0 0 0" xyz="0 0 0.2"/>
             <geometry>
-                <box size="1 0.5 0.1"/>
+                <box size="0.8 0.3 0.1"/>
             </geometry>
         </visual>
@@ -25,5 +25,5 @@
         </visual>
     </link>
-  <joint name="front_joint" type="fixed">
+  <joint name="front_joint_sign" type="fixed">
     <parent link="base_link"/>
     <child link="front"/>
@@ -31,60 +31,60 @@
     <axis xyz="1 0 0"/>
   </joint>
-<!--****************************************-->
-<!--****************************************-->
-    <link name="link_left_f">
-        <visual>
-            <material name="Red">
-                <color rgba="1 0 0 1"/>
-            </material>
-            <origin rpy="0 0 0" xyz="-0.3 0.1 0.1"/>
-            <geometry>
-                <box size="0.05 0.05 0.1"/>
-            </geometry>
-        </visual>
-    </link>
-  <joint name="fixed_left_front" type="fixed">
+<!--*****************REAR STEER***********************-->
+<!--****************************************-->
+    <link name="base_link_rear_steer">
+        <visual>
+            <material name="Red">
+                <color rgba="1 0 0 1"/>
+            </material>
+            <origin rpy="0 0 0" xyz="-0.2 0 0.1"/>
+            <geometry>
+                <box size="0.05 0.1 0.16"/>
+            </geometry>
+        </visual>
+    </link>
+  <joint name="fixed_rear" type="continuous">
     <parent link="base_link"/>
-    <child link="link_left_f"/>
+    <child link="base_link_rear_steer"/>
+    <origin xyz="0 0 0" rpy="0 0 0"/>
+    <axis xyz="0 0 -1"/>
+  </joint>
+<!--****************************************-->
+<!--****************************************-->
+    <link name="rear_steer">
+        <visual>
+            <material name="Red">
+                <color rgba="1 0 0 1"/>
+            </material>
+            <origin rpy="0 0 0" xyz="-0.2 0 0"/>
+            <geometry>
+                <box size="0.05 0.5 0.05"/>
+            </geometry>
+        </visual>
+    </link>
+  <joint name="rear_joint" type="fixed">
+    <parent link="base_link_rear_steer"/>
+    <child link="rear_steer"/>
     <origin xyz="0 0 0" rpy="0 0 0"/>
     <axis xyz="0 0 0"/>
   </joint>
-<!--****************************************-->
-<!--****************************************-->
-    <link name="link_left_f_2">
-        <visual>
-            <material name="Green">
-                <color rgba="0 1 0 1"/>
-            </material>
-            <origin rpy="0 0 0" xyz="-0.2 0.2 0.05"/>
-            <geometry>
-                <box size="0.05 0.2 0.05"/>
-            </geometry>
-        </visual>
-    </link>
-  <joint name="fixed_left_front_2" type="fixed">
-    <parent link="link_left_f"/>
-    <child link="link_left_f_2"/>
-    <origin xyz="0 0 0" rpy="0 0 0"/>
-    <axis xyz="0 0 0"/>
-  </joint>
-<!--****************************************-->
-<!--****************************************-->
-  <link name="left_wheel_f">
-        <visual>
-   	        <material name="Black">
-                <color rgba="0 0 0 1"/>
-            </material>
-             <origin xyz="0 0 0" rpy="1.570795 0 0" />
-            <geometry>
-                <cylinder length="0.15" radius="0.12" />
-            </geometry>
-        </visual>
-    </link>
-<!--****************************************-->
-<!--****************************************-->
-  <joint name="joint_left_wheel_f" type="revolute">
-    <parent link="link_left_f_2"/>
-    <child link="left_wheel_f"/>
+<!--****************REAR WHEELS************************-->
+<!--****************************************-->
+  <link name="left_wheel_rear">
+        <visual>
+   	        <material name="Black">
+                <color rgba="0 0 0 1"/>
+            </material>
+             <origin xyz="0 0 0" rpy="1.570795 0 0" />
+            <geometry>
+                <cylinder length="0.15" radius="0.12" />
+            </geometry>
+        </visual>
+    </link>
+<!--****************************************-->
+<!--****************************************-->
+  <joint name="joint_left_wheel_rear" type="continuous">
+    <parent link="rear_steer"/>
+    <child link="left_wheel_rear"/>
     <origin xyz="-0.20 0.30 0" rpy="0 0 0" />
     <axis xyz="0 1 0" />
@@ -94,4 +94,113 @@
 <!--****************************************-->
 <!--****************************************-->
+<link name="right_wheel_rear">
+        <visual>
+   	        <material name="Black">
+                <color rgba="0 0 0 1"/>
+            </material>
+             <origin xyz="0 0 0" rpy="1.570795 0 0" />
+            <geometry>
+                <cylinder length="0.15" radius="0.12" />
+            </geometry>
+        </visual>
+    </link>
+<!--****************************************-->
+<!--****************************************-->
+  <joint name="joint_right_wheel_rear" type="continuous">
+    <parent link="rear_steer"/>
+    <child link="right_wheel_rear"/>
+    <origin xyz="-0.20 -0.30 0" rpy="0 0 0" />
+    <axis xyz="0 1 0" />
+  <dynamics damping="0.7"/>
+  <limit effort="1000" velocity="0.5" lower="-3.14" upper="3.14" />
+  </joint>
+<!--****************************************-->
+<!--****************************************-->
+<!--*****************FRONT STEER***********************-->
+<!--****************************************-->
+    <link name="base_link_front_steer">
+        <visual>
+            <material name="Red">
+                <color rgba="1 0 0 1"/>
+            </material>
+            <origin rpy="0 0 0" xyz="0.2 0 0.1"/>
+            <geometry>
+                <box size="0.05 0.1 0.16"/>
+            </geometry>
+        </visual>
+    </link>
+  <joint name="fixed_front" type="fixed">
+    <parent link="base_link"/>
+    <child link="base_link_front_steer"/>
+    <origin xyz="0 0 0" rpy="0 0 0"/>
+    <axis xyz="0 0 0"/>
+  </joint>
+<!--****************************************-->
+<!--****************************************-->
+    <link name="front_steer">
+        <visual>
+            <material name="Red">
+                <color rgba="1 0 0 1"/>
+            </material>
+            <origin rpy="0 0 0" xyz="0.2 0 0"/>
+            <geometry>
+                <box size="0.05 0.5 0.05"/>
+            </geometry>
+        </visual>
+    </link>
+  <joint name="front_joint" type="fixed">
+    <parent link="base_link_front_steer"/>
+    <child link="front_steer"/>
+    <origin xyz="0 0 0" rpy="0 0 0"/>
+    <axis xyz="0 0 0"/>
+  </joint>
+<!--****************REAR WHEELS************************-->
+<!--****************************************-->
+  <link name="left_wheel_front">
+        <visual>
+   	        <material name="Black">
+                <color rgba="0 0 0 1"/>
+            </material>
+             <origin xyz="0 0 0" rpy="1.570795 0 0" />
+            <geometry>
+                <cylinder length="0.15" radius="0.12" />
+            </geometry>
+        </visual>
+    </link>
+<!--****************************************-->
+<!--****************************************-->
+  <joint name="joint_left_wheel_front" type="continuous">
+    <parent link="front_steer"/>
+    <child link="left_wheel_front"/>
+    <origin xyz="0.20 0.30 0" rpy="0 0 0" />
+    <axis xyz="0 0 1" />
+  <dynamics damping="0.7"/>
+  <limit effort="1000" velocity="0.5" lower="-3.14" upper="3.14" />
+  </joint>
+<!--****************************************-->
+<!--****************************************-->
+<link name="right_wheel_front">
+        <visual>
+   	        <material name="Black">
+                <color rgba="0 0 0 1"/>
+            </material>
+             <origin xyz="0 0 0" rpy="1.570795 0 0" />
+            <geometry>
+                <cylinder length="0.15" radius="0.12" />
+            </geometry>
+        </visual>
+    </link>
+<!--****************************************-->
+<!--****************************************-->
+  <joint name="joint_right_wheel_front" type="continuous">
+    <parent link="front_steer"/>
+    <child link="right_wheel_front"/>
+    <origin xyz="0.20 -0.30 0" rpy="0 0 0" />
+    <axis xyz="0 0 1" />
+  <dynamics damping="0.7"/>
+  <limit effort="1000" velocity="0.5" lower="-3.14" upper="3.14" />
+  </joint>
+<!--****************************************-->
+<!--****************************************-->
     <link name="sign_left_front">
         <visual>
@@ -106,8 +215,25 @@
     </link>
   <joint name="fixed_sign_left_f" type="fixed">
-    <parent link="left_wheel_f"/>
+    <parent link="left_wheel_rear"/>
     <child link="sign_left_front"/>
     <origin xyz="0 0 0" rpy="0 0 0"/>
     <axis xyz="1 0 0"/>
   </joint>
+    <link name="sign_right_rear">
+        <visual>
+            <material name="White">
+                <color rgba="1 1 1 1"/>
+            </material>
+            <origin rpy="0 0 0" xyz="0 0 0.12"/>
+            <geometry>
+                <sphere radius="0.02" />
+            </geometry>
+        </visual>
+    </link>
+  <joint name="fixed_sign_right_f" type="fixed">
+    <parent link="right_wheel_rear"/>
+    <child link="sign_right_rear"/>
+    <origin xyz="0 0 0" rpy="0 0 0"/>
+    <axis xyz="1 0 0"/>
+  </joint>
 </robot>
